File: Stack-chan_Takao_Base_v121.kicad_sch (KiCad schematic)
At the start: 13 parts, among them CN1 CON_USB-C-6, CN2 CON_GROVE, J1 Conn_01x03, J2 Conn_01x03, SW1 SW_SPDT

Commit message: change USB footprint
Parts:
- CN1: footprint akita:USB-C_6P_V_TH2 -> 74th:Connector_USB-C-Receptacle_TH_6-Pin_Vertical
